File: circuit_schematics/Mercurio_wirelessTransmitter/Mercurio_wirelessTransmitter.sch (KiCad schematic (older format))
At the start: 2 parts

Commit message: Revisada biblioteca de componentes.
Parts:
- removed U?: ATSAM3X8EA-AU, QFP50P2200X2200X145-144N, symbol ATSAM3X8EA-AU:ATSAM3X8EA-AU
- removed U?: CINTERION_PLS83-W, XCVR_CINTERION_PLS83-W, symbol CINTERION_PLS83-W:CINTERION_PLS83-W
- added U?: ATmega8U2-MU, Package_DFN_QFN:QFN-32-1EP_5x5mm_P0.5mm_EP3.1x3.1mm, symbol MCU_Microchip_ATmega:ATmega8U2-MU
Changed lines of the file:
@@
 $EndDescr
 $Comp
-L ATSAM3X8EA-AU:ATSAM3X8EA-AU U?
-U 1 1 62859780
-P 2400 5450
-F 0 "U?" H 2400 10117 50  0000 C CNN
-F 1 "ATSAM3X8EA-AU" H 2400 10026 50  0000 C CNN
-F 2 "QFP50P2200X2200X145-144N" H 2400 5450 50  0001 L BNN
-F 3 "" H 2400 5450 50  0001 L BNN
-F 4 "MICROCHIP" H 2400 5450 50  0001 L BNN "MANUFACTURER"
-F 5 "IPC-7351B" H 2400 5450 50  0001 L BNN "STANDARD"
-F 6 "11057C" H 2400 5450 50  0001 L BNN "PARTREV"
-	1    2400 5450
+L MCU_Microchip_ATmega:ATmega8U2-MU U?
+U 1 1 6286ED92
+P 4200 3750
+F 0 "U?" H 4200 2261 50  0000 C CNN
+F 1 "ATmega8U2-MU" H 4200 2170 50  0000 C CNN
+F 2 "Package_DFN_QFN:QFN-32-1EP_5x5mm_P0.5mm_EP3.1x3.1mm" H 4200 3750 50  0001 C CIN
+F 3 "http://ww1.microchip.com/downloads/en/DeviceDoc/doc7799.pdf" H 4200 3750 50  0001 C CNN
+	1    4200 3750
 	1    0    0    -1
 $EndComp
-$Comp
-L CINTERION_PLS83-W:CINTERION_PLS83-W U?
-U 1 1 6285C9E4
-P 9050 3650
-F 0 "U?" H 9050 5717 50  0000 C CNN
-F 1 "CINTERION_PLS83-W" H 9050 5626 50  0000 C CNN
-F 2 "XCVR_CINTERION_PLS83-W" H 9050 3650 50  0001 L BNN
-F 3 "" H 9050 3650 50  0001 L BNN
-F 4 "Manufacturer Recommendations" H 9050 3650 50  0001 L BNN "STANDARD"
-F 5 "Cinterion" H 9050 3650 50  0001 L BNN "MANUFACTURER"
-F 6 "02.000" H 9050 3650 50  0001 L BNN "PARTREV"
-F 7 "3.32mm" H 9050 3650 50  0001 L BNN "MAXIMUM_PACKAGE_HEIGHT"
-	1    9050 3650
-	1    0    0    -1
-$EndComp
